File: PCB/V1/GeaiRareDit_PCB_Kicad5.kicad_pcb (KiCad board)
At the start: 2 copper layers, 16 parts, among them J1 LIPO_IN, J2 WS2812B_LED_MATRIX, J3 EXT_BUTTONS, Q1 2N3904, Q2 NPD6020P, SW1 Push_1, SW2 Push_2, SW3 Push_3, SW4 Push_4, U1 ITG_MPU6050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

Commit message: Added first version of PCB and CAD designs
Parts:
- removed SW1: Push_1, Button_Switch_THT:SW_PUSH-12mm
- removed SW2: Push_2, Button_Switch_THT:SW_PUSH-12mm
- removed SW3: Push_3, Button_Switch_THT:SW_PUSH-12mm
- removed SW4: Push_4, Button_Switch_THT:SW_PUSH-12mm
- added G***: LOGO, lib_fp:Logo_Papas_Inventeurs_20mm, F.Cu at (115.4, 114.7)
- added G***: LOGO, lib_fp:Logo_Open_Source_Hardware_13mm, F.Cu at (114.4, 81.7)
- added G***: LOGO, lib_fp:Logo_Geai_Rare_15mm_negative, F.Cu at (186.4, 82.2)
- added J4: Conn_SW2, Connector_PinHeader_2.54mm:PinHeader_1x02_P2.54mm_Vertical, F.Cu at (107.8, 129.2)
- added J5: Conn_SW3, Connector_PinHeader_2.54mm:PinHeader_1x02_P2.54mm_Vertical, F.Cu at (194.0, 129.4)
- added J6: Conn_SW4, Connector_PinHeader_2.54mm:PinHeader_1x02_P2.54mm_Vertical, F.Cu at (193.8, 74.1)
- added R3: 470, Resistor_THT:R_Axial_DIN0411_L9.9mm_D3.6mm_P12.70mm_Horizontal, F.Cu at (149.7, 103.0)
- added U1: LiPo_Mngmt_Board, lib_fp:LiPo_Mngmt_Board_Big_Holes, F.Cu at (181.3, 70.6)
- C1: footprint Capacitor_THT:CP_Radial_D12.5mm_P5.00mm -> lib_fp:Edge_CP_Radial_D12.5mm_P5.00mm
- J2: value WS2812B_LED_MATRIX -> Conn_01x11; footprint Connector_PinHeader_2.54mm:PinHeader_1x03_P2.54mm_Horizontal -> Connector_PinHeader_2.54mm:PinHeader_1x11_P2.54mm_Vertical
- J3: value EXT_BUTTONS -> Conn_SW1; footprint Connector_PinHeader_2.54mm:PinHeader_2x04_P2.54mm_Horizontal -> Connector_PinHeader_2.54mm:PinHeader_1x02_P2.54mm_Vertical
- U2: value LiPo_Mngmt_Board -> WS2812B_8x8_matrix; footprint lib_fp:LiPo_Mngmt_Board -> lib_fp:WS2812B_8x8_CJMCU_Matrix; moved to B.Cu
- moved J2 64.7 mm to (145.4, 60.7), turned to 0 degrees
- moved U3 49.8 mm to (136.0, 91.7), turned to 0 degrees
- moved BZ1 40.7 mm to (115.1, 96.3), turned to 180 degrees
- moved C1 26.7 mm to (185.8, 98.5), turned to 0 degrees
- moved uP1 24.8 mm to (138.0, 53.2)
- moved J3 24.2 mm to (108.1, 74.1), turned to 225 degrees
- moved R1 21.8 mm to (122.6, 91.3)
- moved U2 20.4 mm to (186.9, 87.0), turned to 135 degrees
- moved Q1 20.1 mm to (121.8, 100.6), turned to 90 degrees
- moved R2 11.2 mm to (154.4, 103.0), turned to 90 degrees
- moved Q2 9.15 mm to (160.3, 103.4), turned to 0 degrees
- moved J1 7.02 mm to (174.1, 86.1), turned to 270 degrees
- renumbered U1 to U3
Connections:
- J2 pad 2: /WS2812B_DATA_IN -> /RESET
- J2 pad 3: Net-(J2-Pad3) -> /3.3V
- J3 pad 1: GND -> /D2
- Q2 pad 2: Net-(J2-Pad3) -> Net-(Q2-Pad2)
- U2 pad 1: /LIPO+ -> Net-(Q2-Pad2)
- U2 pad 2: /LIPO- -> GND
- U2 pad 3: GND -> Net-(R3-Pad2)
- U2 pad 4: +BATT -> (no net)
- uP1 pad 20: (no net) -> GND
- uP1 pad 21: (no net) -> /RESET
- uP1 pad 22: (no net) -> /3.3V
- uP1 pad 23: (no net) -> /A3
- uP1 pad 24: (no net) -> /A2
- uP1 pad 25: (no net) -> /A1
- uP1 pad 26: (no net) -> /A0
- uP1 pad 27: (no net) -> /D13
- uP1 pad 28: (no net) -> /D12
- uP1 pad 29: (no net) -> /D11
- uP1 pad 30: (no net) -> /D10
Routing:
- net /D4: track 0.00 -> 113.1 mm
- net /D5: track 0.00 -> 103.8 mm
- net Net-(Q2-Pad2): track 0.00 -> 98.2 mm
- net /D3: track 0.00 -> 78.7 mm
- net +BATT: track 0.00 -> 57.3 mm
- net Net-(Q1-Pad3): track 0.00 -> 48.3 mm
- net /I2C_SCL: track 0.00 -> 40.3 mm
- net /WS2812B_DATA_IN: track 0.00 -> 39.2 mm
- net /I2C_SDA: track 0.00 -> 37.5 mm
- net Net-(R3-Pad2): track 0.00 -> 35.3 mm
- net /MPU_VCC: track 0.00 -> 22.0 mm
- net /D2: track 0.00 -> 21.3 mm
- net /BUZZER: track 0.00 -> 18.4 mm
- net /LIPO-: track 0.00 -> 11.3 mm
- net Net-(Q1-Pad2): track 0.00 -> 10.3 mm
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- added copper zone on B.Cu, net +BATT
- added copper zone on F.Cu, net GND
Other:
- board outline added: 99 x 99 mm
- board text added: "Papas Inventeurs GeaiRareDit Janvier 2020"
