File: PCB/V1/_autosave-GeaiRareDit_PCB_Kicad5.sch (KiCad schematic (older format))
At the start: 31 parts, among them J1 LIPO_IN, J2 EXT_BUTTONS, J3 Conn_SW1, J4 Conn_SW2, J5 Conn_SW3, J6 Conn_SW4, Q1 2N3904, Q2 NPD6020P, SW5 RESET_PUSH, U1 LiPo_Mngmt_Board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

Commit message: Added first version of PCB and CAD designs
Parts:
- removed 3.3V1, A0, A1, A2, A3, D10, D11, D12, D13, GND1, RESET1, RX1, TX0: Conn_01x01_Female, Connector_PinHeader_2.54mm:PinHeader_1x01_P2.54mm_Vertical, symbol Connector:Conn_01x01_Female
- removed J2: EXT_BUTTONS, Connector_PinHeader_2.54mm:PinHeader_2x04_P2.54mm_Horizontal, symbol Connector_Generic:Conn_02x04_Counter_Clockwise
- removed SW5: RESET_PUSH, Button_Switch_THT:SW_PUSH_6mm_H5mm, symbol Switch:SW_Push
- added J2: Conn_01x11, Connector_PinHeader_2.54mm:PinHeader_1x11_P2.54mm_Vertical, symbol Connector_Generic:Conn_01x11
- U1: footprint lib_fp:LiPo_Mngmt_Board -> lib_fp:LiPo_Mngmt_Board_Big_Holes
Connections:
- net labels added: 3.3V, A0, A1, A2, A3, D10, D11, D12, D13, RESET
- wire segments 77 -> 64
