File: PCB/V1/GeaiRareDit_PCB_Kicad5.sch (KiCad schematic (older format))
At the start: 18 parts, among them J1 LIPO_IN, J2 WS2812B_LED_MATRIX, J3 EXT_BUTTONS, Q1 2N3904, Q2 NPD6020P, SW1 Push_1, SW2 Push_2, SW3 Push_3, SW4 Push_4, SW5 RESET_PUSH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

Commit message: Added first version of PCB and CAD designs
Parts:
- removed J2: WS2812B_LED_MATRIX, Connector_PinHeader_2.54mm:PinHeader_1x03_P2.54mm_Horizontal, symbol Connector:Conn_01x03_Male
- removed J3: EXT_BUTTONS, Connector_PinHeader_2.54mm:PinHeader_2x04_P2.54mm_Horizontal, symbol Connector_Generic:Conn_02x04_Counter_Clockwise
- removed SW1: Push_1, Button_Switch_THT:SW_PUSH-12mm, symbol Switch:SW_Push
- removed SW2: Push_2, Button_Switch_THT:SW_PUSH-12mm, symbol Switch:SW_Push
- removed SW3: Push_3, Button_Switch_THT:SW_PUSH-12mm, symbol Switch:SW_Push
- removed SW4: Push_4, Button_Switch_THT:SW_PUSH-12mm, symbol Switch:SW_Push
- removed SW5: RESET_PUSH, Button_Switch_THT:SW_PUSH-12mm, symbol Switch:SW_Push
- added J2: Conn_01x11, Connector_PinHeader_2.54mm:PinHeader_1x11_P2.54mm_Vertical, symbol Connector_Generic:Conn_01x11
- added J3: Conn_SW1, Connector_PinHeader_2.54mm:PinHeader_1x02_P2.54mm_Vertical, symbol Connector:Conn_01x02_Male
- added J4: Conn_SW2, Connector_PinHeader_2.54mm:PinHeader_1x02_P2.54mm_Vertical, symbol Connector:Conn_01x02_Male
- added J5: Conn_SW3, Connector_PinHeader_2.54mm:PinHeader_1x02_P2.54mm_Vertical, symbol Connector:Conn_01x02_Male
- added J6: Conn_SW4, Connector_PinHeader_2.54mm:PinHeader_1x02_P2.54mm_Vertical, symbol Connector:Conn_01x02_Male
- added U2: WS2812B_8x8_matrix, lib_fp:WS2812B_8x8_CJMCU_Matrix, symbol Project_Library:WS2812B_8x8_matrix
- C1: footprint Capacitor_THT:CP_Radial_D12.5mm_P5.00mm -> lib_fp:Edge_CP_Radial_D12.5mm_P5.00mm
- renumbered U2 to U1, U1 to U3
Connections:
- net labels added: 3.3V, A0, A1, A2, A3, D10, D11, D12, D13, RESET
- wire segments 61 -> 64
Other:
- moved on the sheet: BZ1, C1, J1, R3, U1, U3, uP1

Commit message: Added several packaging CAD versions and first code configured for Arduino IDE rather than ATOM PlatformIO due to compilation issues
Parts:
- U1: footprint lib_fp:LiPo_Mngmt_Board -> lib_fp:LiPo_Mngmt_Board_Big_Holes
Changed lines of the file:
@@
 F 0 "U1" H 2975 2119 60  0000 C CNN
 F 1 "LiPo_Mngmt_Board" H 2975 2013 60  0000 C CNN
-F 2 "lib_fp:LiPo_Mngmt_Board" H 2950 2600 60  0001 C CNN
+F 2 "lib_fp:LiPo_Mngmt_Board_Big_Holes" H 2950 2600 60  0001 C CNN
 F 3 "" H 2950 2600 60  0000 C CNN
 	1    2950 2600
